File: EM7004-Maho-AxisAdaptor.kicad_pcb (KiCad board)
At the start: 2 copper layers, 41.6 x 119.2 mm, 34 parts, among them J1 1830498, J2 1830498, J3 D-SUB-DR-15PCM-CB, J4 D-SUB-DR-15PCM-CB, J5 DMR-9S, J6 XY2500R-D-5.08-2P, U1 LMR33630ADDAR

Commit message: finalized v0.9.2 design
Parts:
- added J7: S2B-XH-A-1 (LF)(SN), easyeda2kicad:CONN-TH_S2B-XH-A-1-LF-SN, F.Cu at (80.8, 37.4)
- added R5: 0R, Resistor_SMD:R_0603_1608Metric, F.Cu at (83.8, 96.2)
- R1, R2, R4: value 220 -> 680
- R3: value 2k4 -> 4k7
- moved G*** 56.3 mm to (70.1, 91.0)
- moved D1 12.3 mm to (79.5, 44.8)
- moved C3 8.64 mm to (81.0, 52.7)
- moved C4 8.38 mm to (81.0, 60.0)
- moved R1 8.06 mm to (82.6, 44.8), turned to 90 degrees
- moved J5 1.18 mm to (89.9, 89.6)
Routing:
- net 0_Shield: track 99.6 -> 108.2 mm
- net Net-(J4-Pad13): track 17.8 -> 10.1 mm
- net +5V: track 193.0 -> 196.8 mm
- net +24V: track 124.1 -> 120.6 mm
- net 0_Analog-: track 48.2 -> 51.4 mm
- net GND: track 185.2 -> 182.7 mm, vias 80 -> 86
- net 0_Analog+: track 50.9 -> 52.1 mm
- net 1_Analog-: track 54.7 -> 55.8 mm
- net 1_EncoderB: track 36.3 -> 37.1 mm
- net Net-(D1-A): track 2.26 -> 3.06 mm
- net 1_EncoderLatch: track 39.0 -> 38.4 mm
- net Net-(U1-VCC): track 6.59 -> 7.19 mm
- net 1_Analog+: track 51.1 -> 51.7 mm

Commit message: last commit before archiving
Parts:
- added JP0: Latch/Gate-Marker, Jumper:SolderJumper-3_P1.3mm_Bridged12_Pad1.0x1.5mm, F.Cu at (68.3, 110.8)
- added JP1: Latch/Gate-Marker, Jumper:SolderJumper-3_P1.3mm_Bridged12_Pad1.0x1.5mm, F.Cu at (68.3, 67.9)
- moved G*** 8.86 mm to (78.0, 95.1)
- moved G*** 2.03 mm to (76.5, 79.1)
- moved J01 1.34 mm to (88.7, 129.4)
- moved J11 1.34 mm to (88.7, 49.4)
- moved J2 1.17 mm to (88.7, 89.6)
- renumbered J1 to J00, J3 to J01, J2 to J10, J4 to J11, J5 to J2, J6 to J3, J7 to J4
Connections:
- J01 pad 7: 0_EncoderLatch -> 0_Marker
- J11 pad 7: 1_EncoderLatch -> 1_Marker
Routing:
- net 0_Marker: track 0.00 -> 48.6 mm, vias 0 -> 1
- net 1_EncoderLatch: track 38.4 -> 8.47 mm, vias 1 -> 0
- net 1_Marker: track 0.00 -> 26.8 mm, vias 0 -> 1
- net 0_EncoderLatch: track 34.1 -> 8.44 mm
- net 1_EncoderA: track 43.2 -> 62.7 mm
- net 1_EncoderB: track 37.1 -> 56.4 mm
- net GND: track 182.7 -> 169.6 mm, vias 86 -> 89
- net 0_EncoderB: track 36.7 -> 27.3 mm
- net Net-(J01-Pad13): track 24.9 -> 17.1 mm
- net 0_EncoderA: track 39.3 -> 32.4 mm
- net +5V: track 196.8 -> 190.2 mm
- net 0_EncoderGate: track 2.54 -> 8.49 mm
- net 1_EncoderGate: track 2.54 -> 8.46 mm
- net Net-(J11-Pad13): track 10.1 -> 13.6 mm
- net 0_Analog+: track 52.1 -> 49.6 mm
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